Commit message: Made some changes to the urdf file to eliminate the spaces between links

File: urdf_design_project/src/two_joint_robot_description.urdf (robot description, URDF)
Before this commit: robot two_DOF_robot, 4 links, 3 joints
Links:
- link link1: geometry collision box size=0.4 0.4 1.0; visual box size=0.4 0.4 1.0
- link link2: geometry collision cylinder length=1 radius=0.2; visual cylinder length=1 radius=0.2
- link link3: geometry collision cylinder length=1 radius=0.1; visual cylinder length=1 radius=0.1
Joints:
- joint joint2: origin xyz=0 0 2 rpy=0 0 0 -> xyz=0 0 1 rpy=0 0 0
