Commit message: Made some minor changes to numbers to yield better performance

File: trajectory_msgs_project/src/two_DOF_robot_description.urdf (robot description, URDF)
Before this commit: robot two_DOF_robot, 4 links, 3 joints
Links:
- link link2: mass 1 -> 0.5
- link link3: mass 1 -> 0.5

Commit message: More messing around with numbers to get better performance

File: trajectory_msgs_project/src/two_DOF_robot_description.urdf (robot description, URDF)
Before this commit: robot two_DOF_robot, 4 links, 3 joints
Links:
- link link2: mass 0.5 -> 1
- link link3: mass 0.5 -> 1
